Commit message: Modified plugin to use Quaternion and added yaw explitly

File: systems/models/gimbal_small_2d/model.sdf.xacro (robot description, xacro)
@@ -1,13 +1,64 @@
 <?xml version='1.0'?>
 <sdf version='1.6' xmlns:xacro="http://www.ros.org/wiki/xacro">
+  <!-- These match those given in the setup.bash script -->
   <xacro:property name="ros_namespace" value="$(arg ros_namespace)" />
   <xacro:property name="camera_name" value="$(arg camera_name)" />
   <xacro:property name="camera_width" value="$(arg camera_width)" />
   <xacro:property name="camera_height" value="$(arg camera_height)" />
-  <xacro:property name="gimbal_initial_angle" value="$(arg gimbal_initial_angle)" />
+  <xacro:property name="gimbal_initial_pitch" value="$(arg gimbal_initial_pitch)" />
+  <xacro:property name="gimbal_initial_yaw" value="$(arg gimbal_initial_yaw)" />
   <xacro:property name="gimbal_meshes_directory" value="$(arg gimbal_meshes_directory)" />
-    <model name='gimbal_small_2d'>
+  <model name='gimbal_small_2d'>
     <pose>0 0 0.18 0 0 0</pose>
     <link name='base_link'>
+       <inertial>
+        <mass>0.2</mass>
+        <inertia>
+          <ixx>0.0001</ixx>
+          <ixy>0</ixy>
+          <ixz>0</ixz>
+          <iyy>0.0001</iyy>
+          <iyz>0</iyz>
+          <izz>0.0001</izz>
+        </inertia>
+      </inertial>
+      <visual name='base_viz'>
+        <pose>0 0 0.1 1.57 0 0</pose>
+        <geometry>
+         <cylinder>
+            <radius>0.1</radius>
+            <length>0.01</length>
+          </cylinder>
+        </geometry>
+        <material>
+          <script>
+            <uri>file://media/materials/scripts/gazebo.material</uri>
+            <name>Gazebo/FlatBlack</name>
+          </script>
+        </material>
+      </visual>
+      <collision name='base_col'>
+        <pose>0 0 0.1 1.57 0 0</pose>
+        <geometry>
+          <cylinder>
+            <radius>0.1</radius>
+            <length>0.01</length>
+          </cylinder>
+        </geometry>
+        <surface>
+          <friction>
+            <ode>
+              <mu>1</mu>
+              <mu2>1</mu2>
+              <fdir1>0 0 0</fdir1>
+              <slip1>0</slip1>
+              <slip2>0</slip2>
+            </ode>
+          </friction>
+        </surface>
+      </collision>
+    </link>
+    <link name='yaw_base_link'>
+      <pose>0 0 0.18 0 0 0</pose>
        <inertial>
         <mass>0.2</mass>
@@ -164,6 +215,29 @@
       </sensor>
     </link>
+    <joint name='base_joint' type='revolute'>
+       <parent>base_link</parent>
+       <child>yaw_base_link</child>
+      <physics>
+        <ode>
+          <implicit_spring_damper>1</implicit_spring_damper>
+        </ode>
+      </physics>
+      <axis>
+        <xyz>0 0 1</xyz>
+        <dynamics>
+          <damping>0.5</damping>
+        </dynamics>
+        <use_parent_model_frame>1</use_parent_model_frame>
+        <limit>
+          <lower>-0.1</lower>
+          <upper>3.14159265</upper>
+          <effort>10</effort>
+          <velocity>-1</velocity>
+        </limit>
+      </axis>
+      <pose>0 0 0.02 0 0 0</pose>
+    </joint>
     <joint name='tilt_joint' type='revolute'>
-       <parent>base_link</parent>
+       <parent>yaw_base_link</parent>
        <child>tilt_link</child>
       <physics>
@@ -191,6 +265,8 @@
         <namespace>${ros_namespace}</namespace>
       </ros>
+      <!-- Match variables within the controller cpp file -->
       <joint>tilt_joint</joint>
-      <initial_angle>${gimbal_initial_angle}</initial_angle>
+      <initial_pitch>${gimbal_initial_pitch}</initial_pitch>
+      <initial_yaw>${gimbal_initial_yaw}</initial_yaw>
     </plugin>
   </model>

Commit message: Added yaw control and fixed inverted camera

File: systems/models/gimbal_small_2d/model.sdf.xacro (robot description, xacro)
@@ -6,10 +6,12 @@
   <xacro:property name="camera_width" value="$(arg camera_width)" />
   <xacro:property name="camera_height" value="$(arg camera_height)" />
+  <xacro:property name="camera_rotation" value="$(arg camera_rotation)" />
   <xacro:property name="gimbal_initial_pitch" value="$(arg gimbal_initial_pitch)" />
   <xacro:property name="gimbal_initial_yaw" value="$(arg gimbal_initial_yaw)" />
   <xacro:property name="gimbal_meshes_directory" value="$(arg gimbal_meshes_directory)" />
   <model name='gimbal_small_2d'>
-    <pose>0 0 0.18 0 0 0</pose>
+    <pose>0 0 0 0 0 0</pose>
     <link name='base_link'>
+      <pose>0 0 0 0 0 0</pose>
        <inertial>
         <mass>0.2</mass>
@@ -24,8 +26,8 @@
       </inertial>
       <visual name='base_viz'>
-        <pose>0 0 0.1 1.57 0 0</pose>
+        <pose>0 0 0 1.57 0 0</pose>
         <geometry>
          <cylinder>
-            <radius>0.1</radius>
+            <radius>0.11</radius>
             <length>0.01</length>
           </cylinder>
@@ -39,8 +41,8 @@
       </visual>
       <collision name='base_col'>
-        <pose>0 0 0.1 1.57 0 0</pose>
+        <pose>0 0 0 1.57 0 0</pose>
         <geometry>
           <cylinder>
-            <radius>0.1</radius>
+            <radius>0.11</radius>
             <length>0.01</length>
           </cylinder>
@@ -60,5 +62,5 @@
     </link>
     <link name='yaw_base_link'>
-      <pose>0 0 0.18 0 0 0</pose>
+      <pose relative_to="base_joint">-0.015 -0.1 0.025 0 0 0</pose>
        <inertial>
         <mass>0.2</mass>
@@ -121,4 +123,5 @@
     </link>
     <link name='tilt_link'>
+       <pose relative_to="tilt_joint">0 0 -0.005 0 0 0</pose>
        <inertial>
         <mass>0.01</mass>
@@ -180,6 +183,19 @@
         </geometry>
      </collision>
+    </link>
+    <link name="camera_sensor_link">
+      <pose relative_to="camera_joint">0 0 0.03 -1.5707 -1.5707 ${camera_rotation}</pose>
+      <inertial>
+        <mass>0.00001</mass>
+        <inertia>
+          <ixx>0.00001</ixx>
+          <ixy>0</ixy>
+          <ixz>0</ixz>
+          <iyy>0.00001</iyy>
+          <iyz>0</iyz>
+          <izz>0.00001</izz>
+        </inertia>
+      </inertial>
       <sensor name="camera" type="camera">
-        <pose>0 0 0 -1.57 -1.57 0</pose>
         <camera name="head">
           <horizontal_fov>2.0</horizontal_fov>
@@ -224,5 +240,5 @@
       </physics>
       <axis>
-        <xyz>0 0 1</xyz>
+        <xyz>0 1 0</xyz>
         <dynamics>
           <damping>0.5</damping>
@@ -230,11 +246,9 @@
         <use_parent_model_frame>1</use_parent_model_frame>
         <limit>
-          <lower>-0.1</lower>
-          <upper>3.14159265</upper>
           <effort>10</effort>
-          <velocity>-1</velocity>
+          <velocity>1</velocity>
         </limit>
       </axis>
-      <pose>0 0 0.02 0 0 0</pose>
+      <pose relative_to="base_link">0 0 0.0 0 0 0</pose>
     </joint>
     <joint name='tilt_joint' type='revolute'>
@@ -259,5 +273,10 @@
         </limit>
       </axis>
-      <pose>0 0 0.02 0 0 0</pose>
+      <pose relative_to="yaw_base_link">0 0 0.02 0 0 0</pose>
+    </joint>
+    <joint name='camera_joint' type="fixed">
+      <parent>tilt_link</parent>
+      <child>camera_sensor_link</child>
+      <pose relative_to="tilt_link">0.0 0 0 0 0 0</pose>
     </joint>
     <plugin name="gimbal_small_2d" filename="libGimbal2dPlugin.so">
@@ -266,5 +285,6 @@
       </ros>
       <!-- Match variables within the controller cpp file -->
-      <joint>tilt_joint</joint>
+      <pitch_joint>tilt_joint</pitch_joint>
+      <yaw_joint>base_joint</yaw_joint>
       <initial_pitch>${gimbal_initial_pitch}</initial_pitch>
       <initial_yaw>${gimbal_initial_yaw}</initial_yaw>

File: systems/models/gimbal_tripod/model.sdf.xacro (robot description, xacro)
@@ -2,15 +2,16 @@
 <sdf version="1.6" xmlns:xacro='http://ros.org/wiki/xacro'>
   <xacro:property name="ros_namespace" value="$(arg ros_namespace)"/>
-  <model name="iris_demo">
-    <link name="tripod">
+  <xacro:property name="height" value="$(arg height)"/>
+  <model name="gimbal_tripod">
+    <pose>0 0 ${height / 2} 0 0 0</pose>
+    <link name="base">
       <collision name="geom_1">
         <geometry>
-          <box><size>0.5 0.5 1.5 0 0 0</size></box>
+          <box><size>0.5 0.5 ${height} 0 0 0</size></box>
         </geometry>
       </collision>
-      <!-- Keep collision box, but dont show it -->
       <visual name="tripod">
         <geometry>
-          <box><size>0.5 0.5 1.5 0 0 0</size></box>
+          <box><size>0.5 0.5 ${height} 0 0 0</size></box>
         </geometry>
         <material>
@@ -22,17 +23,10 @@
     <include>
       <uri>model://gimbal_small_2d</uri>
-      <pose>0 0 1.0 1.57 0 1.57</pose>
+      <pose relative_to="gimbal_mount">0 0 0.0 1.57 3.14 0.0</pose>
     </include>
-    <joint name="gimbal_mount" type="revolute">
-      <parent>tripod</parent>
+    <joint name="gimbal_mount" type="fixed">
+      <pose relative_to="base">0 0 ${height / 2} 0 0 0</pose>
+      <parent>base</parent>
       <child>gimbal_small_2d::base_link</child>
-      <axis>
-        <limit>
-          <lower>0</lower>
-          <upper>0</upper>
-        </limit>
-        <xyz>0 0 1</xyz>
-        <use_parent_model_frame>true</use_parent_model_frame>
-      </axis>
     </joint>
   </model>
